Commit message: fix(model): 로봇 바퀴 3D 메쉬(mesh) 절대 경로를 패키지 상대 경로로 수정

File: models/limo_ackermann_fortress.urdf (robot description, URDF)
Before this commit: robot limo, 11 links, 10 joints
Links:
- link base_link: geometry collision box size=0.13 0.12 0.1; visual mesh filename=package://limo_capstone/models/meshes/limo_base.dae scale=1 1 1
- link front_left_wheel_link: geometry collision cylinder length=0.045 radius=0.045; visual mesh filename=package://limo_capstone/models/meshes/limo_wheel.dae
- link front_right_wheel_link: geometry collision cylinder length=0.045 radius=0.045; visual mesh filename=package://limo_capstone/models/meshes/limo_wheel.dae
- link rear_left_wheel_link: geometry collision cylinder length=0.045 radius=0.045; visual mesh filename=package://limo_capstone/models/meshes/limo_wheel.dae
- link rear_right_wheel_link: geometry collision cylinder length=0.045 radius=0.045; visual mesh filename=package://limo_capstone/models/meshes/limo_wheel.dae
